File: solar_harvester.sch (EAGLE design)
At the start: 35 parts, among them U1 BQ25505, U2 TPS61322XA, U3 TPS61322XA, U4 MAX17040, U5 INA226

Commit message: uv added schematic
Parts:
- added U6: DMP3085LSD, vrlib_transistor:DMP3085LSD
Connections:
- new net !VB_SEC_ON!: U1.!VB_SEC_ON!, U6.G1, U6.G2
- new net N$15: U6.S1, U6.S2
- new net VCC_P: C11.1, C4.1, C5.1, U1.VOC_SAMP, U1.VSTOR, U6.D2@1, U6.D2@2
- net VCC: now also U6.D1@1, U6.D1@2; no longer C11.1, C4.1, C5.1, U1.VOC_SAMP, U1.VSTOR
Other:
- note added: "UNDER VOLTAGE PROTECTION"
Changed lines of the file:
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@@
 <setting verticaltext="up"/>
 </settings>
-<grid distance="0.1" unitdist="inch" unit="inch" style="lines" multiple="1" display="no" altdistance="0.01" altunitdist="inch" altunit="inch"/>
+<grid distance="1" unitdist="mm" unit="mm" style="lines" multiple="1" display="no" altdistance="0.1" altunitdist="mm" altunit="mm"/>
 <layers>
 <layer number="1" name="Top" color="4" fill="1" visible="no" active="no"/>
@@
 <part name="U$23" library="vrlib_com_symbols" deviceset="VCC" device=""/>
 <part name="U$30" library="vrlib_com_symbols" deviceset="VCC" device=""/>
+<part name="U6" library="vrlib_transistor" deviceset="DMP3085LSD" device=""/>
+<part name="U$5" library="vrlib_com_symbols" deviceset="LOUT" device=""/>
+<part name="U$32" library="vrlib_com_symbols" deviceset="LOUT" device=""/>
+<part name="U$33" library="vrlib_com_symbols" deviceset="VCC" device=""/>
+<part name="U$34" library="vrlib_com_symbols" deviceset="VCC" device=""/>
 </parts>
 <sheets>
@@
 </instance>
 <instance part="U$31" gate="G$1" x="187.278" y="157.48" smashed="yes"/>
+<instance part="U$5" gate="G$1" x="119.634" y="119.38" smashed="yes" rot="R270"/>
 </instances>
 <busses>
@@
 <net name="VCC" class="0">
 <segment>
+<pinref part="L2" gate="G$1" pin="1"/>
+<pinref part="L3" gate="G$1" pin="1"/>
+<wire x1="187.38" y1="150.2" x2="187.38" y2="101.6" width="0.1524" layer="91"/>
+<wire x1="187.38" y1="101.6" x2="187.96" y2="101.6" width="0.1524" layer="91"/>
+<wire x1="187.38" y1="150.2" x2="187.38" y2="157.48" width="0.1524" layer="91"/>
+<junction x="187.38" y="150.2"/>
+<label x="184.712" y="163.02" size="1.778" layer="95"/>
+</segment>
+</net>
+<net name="I2C_SCL" class="0">
+<segment>
+<pinref part="JP1" gate="A" pin="1"/>
+<wire x1="223.52" y1="48.26" x2="213.36" y2="48.26" width="0.1524" layer="91"/>
+<label x="199" y="47.46" size="1.778" layer="95"/>
+</segment>
+</net>
+<net name="!VB_SEC_ON!" class="0">
+<segment>
+<pinref part="U1" gate="G$1" pin="!VB_SEC_ON!"/>
+<wire x1="114.3" y1="119.38" x2="119.38" y2="119.38" width="0.1524" layer="91"/>
+<label x="122.428" y="118.618" size="1.778" layer="95"/>
+</segment>
+</net>
+<net name="VCC_P" class="0">
+<segment>
 <pinref part="C5" gate="G$1" pin="1"/>
 <wire x1="45.224" y1="154.78" x2="43.18" y2="154.78" width="0.1524" layer="91"/>
@@
 <junction x="63.5" y="154.94"/>
 </segment>
-<segment>
-<pinref part="L2" gate="G$1" pin="1"/>
-<pinref part="L3" gate="G$1" pin="1"/>
-<wire x1="187.38" y1="150.2" x2="187.38" y2="101.6" width="0.1524" layer="91"/>
-<wire x1="187.38" y1="101.6" x2="187.96" y2="101.6" width="0.1524" layer="91"/>
-<wire x1="187.38" y1="150.2" x2="187.38" y2="157.48" width="0.1524" layer="91"/>
-<junction x="187.38" y="150.2"/>
-<label x="184.712" y="163.02" size="1.778" layer="95"/>
-</segment>
-</net>
-<net name="I2C_SCL" class="0">
-<segment>
-<pinref part="JP1" gate="A" pin="1"/>
-<wire x1="223.52" y1="48.26" x2="213.36" y2="48.26" width="0.1524" layer="91"/>
-<label x="199" y="47.46" size="1.778" layer="95"/>
-</segment>
 </net>
 </nets>
@@
 Architecture) Research Group</text>
 <text x="217.4" y="10.6" size="1.778" layer="97">Vladislav Rykov</text>
+<wire x1="247.8" y1="92" x2="247.8" y2="38" width="0.1524" layer="97"/>
+<wire x1="247.8" y1="38" x2="156" y2="38" width="0.1524" layer="97"/>
+<wire x1="156" y1="38" x2="156" y2="92" width="0.1524" layer="97"/>
+<wire x1="156" y1="92" x2="247.8" y2="92" width="0.1524" layer="97"/>
+<text x="156" y="93" size="1.778" layer="97">UNDER VOLTAGE PROTECTION</text>
 </plain>
 <instances>
@@
 <instance part="U$23" gate="G$1" x="75.518" y="156.718" smashed="yes"/>
 <instance part="U$30" gate="G$1" x="172.292" y="149.352" smashed="yes"/>
+<instance part="U6" gate="G$1" x="199.58" y="60.96" smashed="yes">
+<attribute name="NAME" x="192.214" y="74.168" size="1.27" layer="95"/>
+<attribute name="VALUE" x="192.214" y="46.482" size="1.27" layer="96"/>
+</instance>
+<instance part="U$32" gate="G$1" x="182.308" y="60.96" smashed="yes" rot="R270"/>
+<instance part="U$33" gate="G$1" x="219.726" y="76.454" smashed="yes"/>
+<instance part="U$34" gate="G$1" x="229.886" y="76.454" smashed="yes"/>
 </instances>
 <busses>
@@
 <junction x="75.584" y="153.282"/>
 <label x="76.962" y="160.528" size="1.778" layer="95"/>
+</segment>
+<segment>
+<pinref part="U6" gate="G$1" pin="D1@1"/>
+<wire x1="209.74" y1="71.12" x2="212.28" y2="71.12" width="0.1524" layer="91"/>
+<wire x1="212.28" y1="71.12" x2="212.28" y2="69.85" width="0.1524" layer="91"/>
+<pinref part="U6" gate="G$1" pin="D1@2"/>
+<wire x1="212.28" y1="69.85" x2="212.28" y2="68.58" width="0.1524" layer="91"/>
+<wire x1="212.28" y1="68.58" x2="209.74" y2="68.58" width="0.1524" layer="91"/>
+<junction x="212.28" y="69.85"/>
+<label x="217.36" y="82.55" size="1.778" layer="95"/>
+<wire x1="212.28" y1="69.85" x2="219.9" y2="69.85" width="0.1524" layer="91"/>
+<wire x1="219.9" y1="69.85" x2="219.9" y2="76.2" width="0.1524" layer="91"/>
 </segment>
 </net>
@@
 </segment>
 </net>
+<net name="VCC_P" class="0">
+<segment>
+<pinref part="U6" gate="G$1" pin="D2@1"/>
+<wire x1="209.74" y1="53.34" x2="212.28" y2="53.34" width="0.1524" layer="91"/>
+<pinref part="U6" gate="G$1" pin="D2@2"/>
+<wire x1="212.28" y1="53.34" x2="212.28" y2="52.07" width="0.1524" layer="91"/>
+<wire x1="212.28" y1="52.07" x2="212.28" y2="50.8" width="0.1524" layer="91"/>
+<wire x1="212.28" y1="50.8" x2="209.74" y2="50.8" width="0.1524" layer="91"/>
+<junction x="212.28" y="52.07"/>
+<label x="227.52" y="82.55" size="1.778" layer="95"/>
+<wire x1="212.28" y1="52.07" x2="230.06" y2="52.07" width="0.1524" layer="91"/>
+<wire x1="230.06" y1="52.07" x2="230.06" y2="76.2" width="0.1524" layer="91"/>
+</segment>
+</net>
+<net name="N$15" class="0">
+<segment>
+<pinref part="U6" gate="G$1" pin="S2"/>
+<wire x1="209.74" y1="58.42" x2="212.28" y2="58.42" width="0.1524" layer="91"/>
+<wire x1="212.28" y1="58.42" x2="212.28" y2="63.5" width="0.1524" layer="91"/>
+<pinref part="U6" gate="G$1" pin="S1"/>
+<wire x1="212.28" y1="63.5" x2="209.74" y2="63.5" width="0.1524" layer="91"/>
+</segment>
+</net>
+<net name="!VB_SEC_ON!" class="0">
+<segment>
+<pinref part="U6" gate="G$1" pin="G1"/>
+<pinref part="U6" gate="G$1" pin="G2"/>
+<wire x1="189.42" y1="63.5" x2="189.42" y2="60.96" width="0.1524" layer="91"/>
+<wire x1="189.42" y1="60.96" x2="189.42" y2="58.42" width="0.1524" layer="91"/>
+<wire x1="189.42" y1="60.96" x2="184.34" y2="60.96" width="0.1524" layer="91"/>
+<junction x="189.42" y="60.96"/>
+<label x="166.56" y="59.944" size="1.778" layer="95"/>
+</segment>
+</net>

Commit message: uv routed done
Other:
- moved on the sheet: U6
Changed lines of the file:
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@@
 Architecture) Research Group</text>
 <text x="217.4" y="10.6" size="1.778" layer="97">Vladislav Rykov</text>
-<wire x1="247.8" y1="92" x2="247.8" y2="38" width="0.1524" layer="97"/>
-<wire x1="247.8" y1="38" x2="156" y2="38" width="0.1524" layer="97"/>
-<wire x1="156" y1="38" x2="156" y2="92" width="0.1524" layer="97"/>
-<wire x1="156" y1="92" x2="247.8" y2="92" width="0.1524" layer="97"/>
-<text x="156" y="93" size="1.778" layer="97">UNDER VOLTAGE PROTECTION</text>
+<wire x1="247.8" y1="88" x2="247.8" y2="34" width="0.1524" layer="97"/>
+<wire x1="247.8" y1="34" x2="156" y2="34" width="0.1524" layer="97"/>
+<wire x1="156" y1="34" x2="156" y2="88" width="0.1524" layer="97"/>
+<wire x1="156" y1="88" x2="247.8" y2="88" width="0.1524" layer="97"/>
+<text x="156" y="89" size="1.778" layer="97">UNDER VOLTAGE PROTECTION</text>
 </plain>
 <instances>
@@
 <instance part="U$23" gate="G$1" x="75.518" y="156.718" smashed="yes"/>
 <instance part="U$30" gate="G$1" x="172.292" y="149.352" smashed="yes"/>
-<instance part="U6" gate="G$1" x="199.58" y="60.96" smashed="yes">
-<attribute name="NAME" x="192.214" y="74.168" size="1.27" layer="95"/>
-<attribute name="VALUE" x="192.214" y="46.482" size="1.27" layer="96"/>
-</instance>
-<instance part="U$32" gate="G$1" x="182.308" y="60.96" smashed="yes" rot="R270"/>
-<instance part="U$33" gate="G$1" x="219.726" y="76.454" smashed="yes"/>
-<instance part="U$34" gate="G$1" x="229.886" y="76.454" smashed="yes"/>
+<instance part="U6" gate="G$1" x="199.58" y="56.96" smashed="yes">
+<attribute name="NAME" x="192.214" y="70.168" size="1.27" layer="95"/>
+<attribute name="VALUE" x="192.214" y="42.482" size="1.27" layer="96"/>
+</instance>
+<instance part="U$32" gate="G$1" x="182.308" y="56.96" smashed="yes" rot="R270"/>
+<instance part="U$33" gate="G$1" x="219.726" y="72.454" smashed="yes"/>
+<instance part="U$34" gate="G$1" x="229.886" y="72.454" smashed="yes"/>
 </instances>
 <busses>
@@
 <segment>
 <pinref part="U6" gate="G$1" pin="D1@1"/>
-<wire x1="209.74" y1="71.12" x2="212.28" y2="71.12" width="0.1524" layer="91"/>
-<wire x1="212.28" y1="71.12" x2="212.28" y2="69.85" width="0.1524" layer="91"/>
+<wire x1="209.74" y1="67.12" x2="212.28" y2="67.12" width="0.1524" layer="91"/>
+<wire x1="212.28" y1="67.12" x2="212.28" y2="65.85" width="0.1524" layer="91"/>
 <pinref part="U6" gate="G$1" pin="D1@2"/>
-<wire x1="212.28" y1="69.85" x2="212.28" y2="68.58" width="0.1524" layer="91"/>
-<wire x1="212.28" y1="68.58" x2="209.74" y2="68.58" width="0.1524" layer="91"/>
-<junction x="212.28" y="69.85"/>
-<label x="217.36" y="82.55" size="1.778" layer="95"/>
-<wire x1="212.28" y1="69.85" x2="219.9" y2="69.85" width="0.1524" layer="91"/>
-<wire x1="219.9" y1="69.85" x2="219.9" y2="76.2" width="0.1524" layer="91"/>
+<wire x1="212.28" y1="65.85" x2="212.28" y2="64.58" width="0.1524" layer="91"/>
+<wire x1="212.28" y1="64.58" x2="209.74" y2="64.58" width="0.1524" layer="91"/>
+<junction x="212.28" y="65.85"/>
+<label x="217.36" y="78.55" size="1.778" layer="95"/>
+<wire x1="212.28" y1="65.85" x2="219.9" y2="65.85" width="0.1524" layer="91"/>
+<wire x1="219.9" y1="65.85" x2="219.9" y2="72.2" width="0.1524" layer="91"/>
 </segment>
 </net>
@@
 <segment>
 <pinref part="U6" gate="G$1" pin="D2@1"/>
-<wire x1="209.74" y1="53.34" x2="212.28" y2="53.34" width="0.1524" layer="91"/>
+<wire x1="209.74" y1="49.34" x2="212.28" y2="49.34" width="0.1524" layer="91"/>
 <pinref part="U6" gate="G$1" pin="D2@2"/>
-<wire x1="212.28" y1="53.34" x2="212.28" y2="52.07" width="0.1524" layer="91"/>
-<wire x1="212.28" y1="52.07" x2="212.28" y2="50.8" width="0.1524" layer="91"/>
-<wire x1="212.28" y1="50.8" x2="209.74" y2="50.8" width="0.1524" layer="91"/>
-<junction x="212.28" y="52.07"/>
-<label x="227.52" y="82.55" size="1.778" layer="95"/>
-<wire x1="212.28" y1="52.07" x2="230.06" y2="52.07" width="0.1524" layer="91"/>
-<wire x1="230.06" y1="52.07" x2="230.06" y2="76.2" width="0.1524" layer="91"/>
+<wire x1="212.28" y1="49.34" x2="212.28" y2="48.07" width="0.1524" layer="91"/>
+<wire x1="212.28" y1="48.07" x2="212.28" y2="46.8" width="0.1524" layer="91"/>
+<wire x1="212.28" y1="46.8" x2="209.74" y2="46.8" width="0.1524" layer="91"/>
+<junction x="212.28" y="48.07"/>
+<label x="227.52" y="78.55" size="1.778" layer="95"/>
+<wire x1="212.28" y1="48.07" x2="230.06" y2="48.07" width="0.1524" layer="91"/>
+<wire x1="230.06" y1="48.07" x2="230.06" y2="72.2" width="0.1524" layer="91"/>
 </segment>
 </net>
@@
 <segment>
 <pinref part="U6" gate="G$1" pin="S2"/>
-<wire x1="209.74" y1="58.42" x2="212.28" y2="58.42" width="0.1524" layer="91"/>
-<wire x1="212.28" y1="58.42" x2="212.28" y2="63.5" width="0.1524" layer="91"/>
+<wire x1="209.74" y1="54.42" x2="212.28" y2="54.42" width="0.1524" layer="91"/>
+<wire x1="212.28" y1="54.42" x2="212.28" y2="59.5" width="0.1524" layer="91"/>
 <pinref part="U6" gate="G$1" pin="S1"/>
-<wire x1="212.28" y1="63.5" x2="209.74" y2="63.5" width="0.1524" layer="91"/>
+<wire x1="212.28" y1="59.5" x2="209.74" y2="59.5" width="0.1524" layer="91"/>
 </segment>
 </net>
@@
 <pinref part="U6" gate="G$1" pin="G1"/>
 <pinref part="U6" gate="G$1" pin="G2"/>
-<wire x1="189.42" y1="63.5" x2="189.42" y2="60.96" width="0.1524" layer="91"/>
-<wire x1="189.42" y1="60.96" x2="189.42" y2="58.42" width="0.1524" layer="91"/>
-<wire x1="189.42" y1="60.96" x2="184.34" y2="60.96" width="0.1524" layer="91"/>
-<junction x="189.42" y="60.96"/>
-<label x="166.56" y="59.944" size="1.778" layer="95"/>
-</segment>
-</net>
+<wire x1="189.42" y1="59.5" x2="189.42" y2="56.96" width="0.1524" layer="91"/>
+<wire x1="189.42" y1="56.96" x2="189.42" y2="54.42" width="0.1524" layer="91"/>
+<wire x1="189.42" y1="56.96" x2="184.34" y2="56.96" width="0.1524" layer="91"/>
+<junction x="189.42" y="56.96"/>
+<label x="166.56" y="55.944" size="1.778" layer="95"/>
+</segment>
+</net>
