File: solar_harvester.sch (EAGLE design)
At the start: 36 parts, among them U1 BQ25505, U2 TPS61322XA, U3 TPS61322XA, U4 MAX17040, U5 INA226, U6 DMP3085LSD

Commit message: tps, fids added, todo:rev gnd, pass grc
Parts:
- added FID1, U$36: FIDUCIAL_50, vrlib_prod:FIDUCIAL_50
- added TP1, TP2, TP3, TP4, TP5, TP6: TPTP10SQ, testpad:TPTP10SQ
Connections:
- net GND: now also TP2.TP
- net PVIN_AN: now also TP1.TP
- net VCC: now also TP4.TP
- net VDD3V3: now also TP5.TP
- net VDD5: now also TP6.TP
- net VIN_BAT: now also TP3.TP
Changed lines of the file:
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@@
 <part name="U$33" library="vrlib_com_symbols" deviceset="VCC" device=""/>
 <part name="U$34" library="vrlib_com_symbols" deviceset="VCC" device=""/>
+<part name="TP1" library="testpad" library_urn="urn:adsk.eagle:library:385" deviceset="TP" device="TP10SQ" package3d_urn="urn:adsk.eagle:package:27962/1"/>
+<part name="TP2" library="testpad" library_urn="urn:adsk.eagle:library:385" deviceset="TP" device="TP10SQ" package3d_urn="urn:adsk.eagle:package:27962/1"/>
+<part name="TP3" library="testpad" library_urn="urn:adsk.eagle:library:385" deviceset="TP" device="TP10SQ" package3d_urn="urn:adsk.eagle:package:27962/1"/>
+<part name="TP4" library="testpad" library_urn="urn:adsk.eagle:library:385" deviceset="TP" device="TP10SQ" package3d_urn="urn:adsk.eagle:package:27962/1"/>
+<part name="TP5" library="testpad" library_urn="urn:adsk.eagle:library:385" deviceset="TP" device="TP10SQ" package3d_urn="urn:adsk.eagle:package:27962/1"/>
+<part name="TP6" library="testpad" library_urn="urn:adsk.eagle:library:385" deviceset="TP" device="TP10SQ" package3d_urn="urn:adsk.eagle:package:27962/1"/>
+<part name="FID1" library="vrlib_prod" deviceset="FIDUCIAL_50" device=""/>
+<part name="U$36" library="vrlib_prod" deviceset="FIDUCIAL_50" device=""/>
 </parts>
 <sheets>
@@
 <instance part="U$31" gate="G$1" x="187.278" y="157.48" smashed="yes"/>
 <instance part="U$5" gate="G$1" x="119.634" y="119.38" smashed="yes" rot="R270"/>
+<instance part="TP1" gate="G$1" x="137.16" y="160.02" smashed="yes">
+<attribute name="NAME" x="131.572" y="160.274" size="1.778" layer="95"/>
+<attribute name="TP_SIGNAL_NAME" x="138.43" y="158.75" size="1.778" layer="97"/>
+</instance>
+<instance part="TP2" gate="G$1" x="38.1" y="152.4" smashed="yes">
+<attribute name="NAME" x="35.56" y="152.908" size="1.778" layer="95"/>
+<attribute name="TP_SIGNAL_NAME" x="39.37" y="151.13" size="1.778" layer="97"/>
+</instance>
+<instance part="TP3" gate="G$1" x="18.034" y="137.16" smashed="yes" rot="R180">
+<attribute name="NAME" x="19.304" y="136.398" size="1.778" layer="95" rot="R180"/>
+<attribute name="TP_SIGNAL_NAME" x="16.764" y="138.43" size="1.778" layer="97" rot="R180"/>
+</instance>
+<instance part="TP5" gate="G$1" x="124.46" y="48.26" smashed="yes">
+<attribute name="NAME" x="121.92" y="48.768" size="1.778" layer="95"/>
+<attribute name="TP_SIGNAL_NAME" x="125.73" y="46.99" size="1.778" layer="97"/>
+</instance>
+<instance part="TP6" gate="G$1" x="170.18" y="48.26" smashed="yes">
+<attribute name="NAME" x="167.64" y="48.768" size="1.778" layer="95"/>
+<attribute name="TP_SIGNAL_NAME" x="171.45" y="46.99" size="1.778" layer="97"/>
+</instance>
+<instance part="FID1" gate="G$1" x="71.12" y="12.7" smashed="yes">
+<attribute name="NAME" x="68.072" y="18.288" size="1.27" layer="95"/>
+</instance>
+<instance part="U$36" gate="G$1" x="83.82" y="12.7" smashed="yes">
+<attribute name="NAME" x="80.772" y="18.288" size="1.27" layer="95"/>
+</instance>
 </instances>
 <busses>
@@
 <pinref part="C5" gate="G$1" pin="2"/>
 <wire x1="22.686" y1="147.828" x2="25.4" y2="147.828" width="0.1524" layer="91"/>
-<wire x1="25.4" y1="147.828" x2="45.224" y2="147.828" width="0.1524" layer="91"/>
+<wire x1="25.4" y1="147.828" x2="38.1" y2="147.828" width="0.1524" layer="91"/>
+<wire x1="38.1" y1="147.828" x2="45.224" y2="147.828" width="0.1524" layer="91"/>
 <wire x1="45.224" y1="147.828" x2="45.224" y2="148.176" width="0.1524" layer="91"/>
 <pinref part="C11" gate="G$1" pin="2"/>
@@
 <pinref part="C4" gate="G$1" pin="2"/>
 <junction x="52.302" y="148.018"/>
+<pinref part="TP2" gate="G$1" pin="TP"/>
+<wire x1="38.1" y1="147.828" x2="38.1" y2="149.86" width="0.1524" layer="91"/>
+<junction x="38.1" y="147.828"/>
 </segment>
 </net>
@@
 <pinref part="BAT_IN" gate="G$1" pin="VIN"/>
 <wire x1="48.006" y1="143.002" x2="33.02" y2="143.002" width="0.1524" layer="91"/>
-<wire x1="33.02" y1="143.002" x2="17.606" y2="143.002" width="0.1524" layer="91"/>
+<wire x1="33.02" y1="143.002" x2="18.034" y2="143.002" width="0.1524" layer="91"/>
+<wire x1="18.034" y1="143.002" x2="17.606" y2="143.002" width="0.1524" layer="91"/>
 <wire x1="17.606" y1="143.002" x2="17.606" y2="147.828" width="0.1524" layer="91"/>
 <junction x="48.006" y="143.002"/>
 <wire x1="33.02" y1="143.002" x2="33.02" y2="157.48" width="0.1524" layer="91"/>
 <label x="27.94" y="160.274" size="1.778" layer="95"/>
+<pinref part="TP3" gate="G$1" pin="TP"/>
+<wire x1="18.034" y1="143.002" x2="18.034" y2="139.7" width="0.1524" layer="91"/>
+<junction x="18.034" y="143.002"/>
 </segment>
 </net>
@@
 <wire x1="157.48" y1="43.18" x2="157.48" y2="38.1" width="0.1524" layer="91"/>
 <label x="154.94" y="33.02" size="1.778" layer="95"/>
+<pinref part="TP6" gate="G$1" pin="TP"/>
+<wire x1="157.48" y1="38.1" x2="170.18" y2="38.1" width="0.1524" layer="91"/>
+<wire x1="170.18" y1="38.1" x2="170.18" y2="45.72" width="0.1524" layer="91"/>
 </segment>
 </net>
@@
 <wire x1="132.08" y1="43.18" x2="132.08" y2="38.1" width="0.1524" layer="91"/>
 <label x="127" y="33.02" size="1.778" layer="95"/>
+<pinref part="TP5" gate="G$1" pin="TP"/>
+<wire x1="124.46" y1="45.72" x2="124.46" y2="38.1" width="0.1524" layer="91"/>
+<wire x1="124.46" y1="38.1" x2="132.08" y2="38.1" width="0.1524" layer="91"/>
+<junction x="132.08" y="38.1"/>
 </segment>
 </net>
@@
 <wire x1="114.3" y1="132.08" x2="142.24" y2="132.08" width="0.1524" layer="91"/>
 <wire x1="142.24" y1="132.08" x2="142.24" y2="154.94" width="0.1524" layer="91"/>
-<wire x1="142.24" y1="154.94" x2="134.62" y2="154.94" width="0.1524" layer="91"/>
+<wire x1="142.24" y1="154.94" x2="137.16" y2="154.94" width="0.1524" layer="91"/>
 <junction x="134.62" y="154.94"/>
-<label x="143.764" y="162.052" size="1.778" layer="95" rot="R180"/>
+<label x="150.622" y="162.052" size="1.778" layer="95" rot="R180"/>
+<wire x1="137.16" y1="154.94" x2="134.62" y2="154.94" width="0.1524" layer="91"/>
 <wire x1="142.24" y1="154.94" x2="142.24" y2="157.48" width="0.1524" layer="91"/>
 <junction x="142.24" y="154.94"/>
@@
 <wire x1="142.24" y1="154.94" x2="142.24" y2="154.956" width="0.1524" layer="91"/>
 <wire x1="142.24" y1="154.956" x2="144.382" y2="154.956" width="0.1524" layer="91"/>
+<pinref part="TP1" gate="G$1" pin="TP"/>
+<wire x1="137.16" y1="157.48" x2="137.16" y2="154.94" width="0.1524" layer="91"/>
+<junction x="137.16" y="154.94"/>
 </segment>
 </net>
@@
 <instance part="U$33" gate="G$1" x="219.726" y="72.454" smashed="yes"/>
 <instance part="U$34" gate="G$1" x="229.886" y="72.454" smashed="yes"/>
+<instance part="TP4" gate="G$1" x="85.598" y="159.512" smashed="yes">
+<attribute name="NAME" x="86.868" y="160.274" size="1.778" layer="95"/>
+<attribute name="TP_SIGNAL_NAME" x="86.868" y="158.242" size="1.778" layer="97"/>
+</instance>
 </instances>
 <busses>
@@
 <junction x="75.584" y="153.282"/>
 <label x="76.962" y="160.528" size="1.778" layer="95"/>
-</segment>
-<segment>
+<pinref part="TP4" gate="G$1" pin="TP"/>
+<wire x1="75.584" y1="153.282" x2="85.598" y2="153.282" width="0.1524" layer="91"/>
+<wire x1="85.598" y1="153.282" x2="85.598" y2="156.972" width="0.1524" layer="91"/>
+</segment>
+<segment>
